File: project-nixie-v1.brd (EAGLE design)
At the start: 22.9 x 54.6 mm, 8 parts, among them J1 D

Commit message: version 2 of the board
Parts:
- removed E$1: (no value), holes:3,0-PAD
- added U$1: (no value), holes:3,0
- moved NX 36.9 mm to (8.89, -10.2), turned to 0 degrees
- moved DOTS 18.1 mm to (1.91, 24.8), turned to 270 degrees
- moved J1 11.7 mm to (8.26, 31.1)
- moved PWR 10.8 mm to (1.91, 31.1)
- moved R1 9.69 mm to (19.7, 19.7), turned to 90 degrees
- moved A 5.75 mm to (19.7, 31.1)
- moved DRIVER 0.90 mm to (10.8, 5.71)
Routing:
- net D: track 57.3 -> 37.2 mm, vias 1 -> 2
- net N$10: track 22.3 -> 41.9 mm
- net N$12: track 24.3 -> 7.62 mm, vias 1 -> 0
- net 5V: track 48.2 -> 63.5 mm
- net N$1: track 26.1 -> 40.3 mm, vias 0 -> 1
- net GND: track 43.3 -> 29.6 mm, vias 0 -> 1
- net LHDP: track 10.2 -> 21.4 mm, vias 0 -> 1
- net N$8: track 26.6 -> 17.3 mm
- net N$9: track 27.4 -> 18.4 mm
- net N$6: track 14.1 -> 7.43 mm, vias 1 -> 0
- net N$11: track 19.8 -> 13.2 mm
- net N$2: track 26.0 -> 32.5 mm, vias 1 -> 0
- net N$4: track 12.7 -> 7.27 mm
- net B: track 45.3 -> 50.6 mm, vias 1 -> 3
- net N$7: track 16.8 -> 21.5 mm
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Other:
- board size 22.9 x 54.6 mm -> 22.9 x 43.2 mm
- board text added: "A"
- board text added: "Nixie Board"
- board text added: "P. M. Canseco"
- board text added: "n"
- board text removed: "5V"
- board text removed: "P.M.CANSECO"
