File: project-nixie.sch (EAGLE design)
At the start: 8 parts, among them J1 D

Commit message: re-upload to seeed
Parts:
- removed FRAME1: FRAME-LETTER, SparkFun-Aesthetics:FRAME-LETTER
Other:
- moved on the sheet: DRIVERP
Changed lines of the file:
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@@
 <grid distance="0.1" unitdist="inch" unit="inch" style="lines" multiple="1" display="no" altdistance="0.01" altunitdist="inch" altunit="inch"/>
 <layers>
-<layer number="1" name="Top" color="4" fill="1" visible="yes" active="no"/>
-<layer number="16" name="Bottom" color="1" fill="1" visible="yes" active="no"/>
-<layer number="17" name="Pads" color="2" fill="1" visible="yes" active="no"/>
-<layer number="18" name="Vias" color="2" fill="1" visible="yes" active="no"/>
-<layer number="19" name="Unrouted" color="6" fill="1" visible="yes" active="no"/>
-<layer number="20" name="Dimension" color="15" fill="1" visible="yes" active="no"/>
-<layer number="21" name="tPlace" color="7" fill="1" visible="yes" active="no"/>
-<layer number="22" name="bPlace" color="7" fill="1" visible="yes" active="no"/>
-<layer number="23" name="tOrigins" color="15" fill="1" visible="yes" active="no"/>
-<layer number="24" name="bOrigins" color="15" fill="1" visible="yes" active="no"/>
-<layer number="25" name="tNames" color="7" fill="1" visible="yes" active="no"/>
-<layer number="26" name="bNames" color="7" fill="1" visible="yes" active="no"/>
-<layer number="27" name="tValues" color="7" fill="1" visible="yes" active="no"/>
-<layer number="28" name="bValues" color="7" fill="1" visible="yes" active="no"/>
+<layer number="1" name="Top" color="4" fill="1" visible="no" active="no"/>
+<layer number="16" name="Bottom" color="1" fill="1" visible="no" active="no"/>
+<layer number="17" name="Pads" color="2" fill="1" visible="no" active="no"/>
+<layer number="18" name="Vias" color="2" fill="1" visible="no" active="no"/>
+<layer number="19" name="Unrouted" color="6" fill="1" visible="no" active="no"/>
+<layer number="20" name="Dimension" color="15" fill="1" visible="no" active="no"/>
+<layer number="21" name="tPlace" color="7" fill="1" visible="no" active="no"/>
+<layer number="22" name="bPlace" color="7" fill="1" visible="no" active="no"/>
+<layer number="23" name="tOrigins" color="15" fill="1" visible="no" active="no"/>
+<layer number="24" name="bOrigins" color="15" fill="1" visible="no" active="no"/>
+<layer number="25" name="tNames" color="7" fill="1" visible="no" active="no"/>
+<layer number="26" name="bNames" color="7" fill="1" visible="no" active="no"/>
+<layer number="27" name="tValues" color="7" fill="1" visible="no" active="no"/>
+<layer number="28" name="bValues" color="7" fill="1" visible="no" active="no"/>
 <layer number="29" name="tStop" color="15" fill="3" visible="no" active="no"/>
 <layer number="30" name="bStop" color="7" fill="6" visible="no" active="no"/>
@@
 <layer number="35" name="tGlue" color="7" fill="4" visible="no" active="no"/>
 <layer number="36" name="bGlue" color="7" fill="5" visible="no" active="no"/>
-<layer number="37" name="tTest" color="7" fill="1" visible="yes" active="no"/>
-<layer number="38" name="bTest" color="7" fill="1" visible="yes" active="no"/>
+<layer number="37" name="tTest" color="7" fill="1" visible="no" active="no"/>
+<layer number="38" name="bTest" color="7" fill="1" visible="no" active="no"/>
 <layer number="39" name="tKeepout" color="4" fill="11" visible="no" active="no"/>
 <layer number="40" name="bKeepout" color="1" fill="11" visible="no" active="no"/>
@@
 <layer number="44" name="Drills" color="7" fill="1" visible="no" active="no"/>
 <layer number="45" name="Holes" color="7" fill="1" visible="no" active="no"/>
-<layer number="46" name="Milling" color="3" fill="1" visible="yes" active="no"/>
-<layer number="47" name="Measures" color="7" fill="1" visible="yes" active="no"/>
-<layer number="48" name="Document" color="7" fill="1" visible="yes" active="no"/>
-<layer number="49" name="Reference" color="13" fill="1" visible="yes" active="no"/>
-<layer number="50" name="dxf" color="7" fill="1" visible="yes" active="no"/>
-<layer number="51" name="tDocu" color="14" fill="1" visible="yes" active="no"/>
-<layer number="52" name="bDocu" color="7" fill="1" visible="yes" active="no"/>
-<layer number="53" name="tGND_GNDA" color="7" fill="9" visible="yes" active="no"/>
-<layer number="54" name="bGND_GNDA" color="1" fill="9" visible="yes" active="no"/>
-<layer number="56" name="wert" color="7" fill="1" visible="yes" active="no"/>
-<layer number="57" name="tCAD" color="7" fill="1" visible="yes" active="no"/>
-<layer number="59" name="tCarbon" color="7" fill="1" visible="yes" active="no"/>
-<layer number="60" name="bCarbon" color="7" fill="1" visible="yes" active="no"/>
+<layer number="46" name="Milling" color="3" fill="1" visible="no" active="no"/>
+<layer number="47" name="Measures" color="7" fill="1" visible="no" active="no"/>
+<layer number="48" name="Document" color="7" fill="1" visible="no" active="no"/>
+<layer number="49" name="Reference" color="13" fill="1" visible="no" active="no"/>
+<layer number="50" name="dxf" color="7" fill="1" visible="no" active="no"/>
+<layer number="51" name="tDocu" color="14" fill="1" visible="no" active="no"/>
+<layer number="52" name="bDocu" color="7" fill="1" visible="no" active="no"/>
+<layer number="53" name="tGND_GNDA" color="7" fill="9" visible="no" active="no"/>
+<layer number="54" name="bGND_GNDA" color="1" fill="9" visible="no" active="no"/>
+<layer number="56" name="wert" color="7" fill="1" visible="no" active="no"/>
+<layer number="57" name="tCAD" color="7" fill="1" visible="no" active="no"/>
+<layer number="59" name="tCarbon" color="7" fill="1" visible="no" active="no"/>
+<layer number="60" name="bCarbon" color="7" fill="1" visible="no" active="no"/>
 <layer number="90" name="Modules" color="5" fill="1" visible="yes" active="yes"/>
 <layer number="91" name="Nets" color="2" fill="1" visible="yes" active="yes"/>
@@
 </classes>
 <parts>
-<part name="FRAME1" library="SparkFun-Aesthetics" deviceset="FRAME-LETTER" device=""/>
 <part name="N1" library="russian-nixies" deviceset="IN-16" device=""/>
 <part name="DRIVER" library="74xx-us" deviceset="74*141" device="N"/>
@@
 </plain>
 <instances>
-<instance part="FRAME1" gate="G$1" x="-1549.4" y="680.72"/>
-<instance part="FRAME1" gate="V" x="-1402.08" y="680.72"/>
 <instance part="N1" gate="G$1" x="-1432.56" y="797.56"/>
 <instance part="DRIVER" gate="A" x="-1465.58" y="802.64"/>
@@
 <instance part="DOTS" gate="G$1" x="-1414.78" y="822.96" rot="R270"/>
 <instance part="A" gate="G$1" x="-1381.76" y="797.56" rot="MR0"/>
-<instance part="DRIVER" gate="P" x="-1465.58" y="825.5" rot="R90"/>
+<instance part="DRIVER" gate="P" x="-1465.58" y="822.96" smashed="yes" rot="R90">
+<attribute name="NAME" x="-1459.865" y="829.945" size="1.778" layer="95" rot="R180"/>
+</instance>
 <instance part="PWR" gate="G$1" x="-1468.12" y="843.28" rot="R270"/>
 <instance part="J1" gate="G$1" x="-1503.68" y="800.1"/>
@@
 <segment>
 <pinref part="DRIVER" gate="P" pin="VCC"/>
-<wire x1="-1475.74" y1="825.5" x2="-1478.28" y2="825.5" width="0.1524" layer="91"/>
+<wire x1="-1475.74" y1="822.96" x2="-1478.28" y2="825.5" width="0.1524" layer="91"/>
 <wire x1="-1478.28" y1="825.5" x2="-1478.28" y2="833.12" width="0.1524" layer="91"/>
 <pinref part="PWR" gate="G$1" pin="1"/>
 <wire x1="-1478.28" y1="833.12" x2="-1468.12" y2="833.12" width="0.1524" layer="91"/>
 <wire x1="-1468.12" y1="833.12" x2="-1468.12" y2="835.66" width="0.1524" layer="91"/>
+<label x="-1478.28" y="828.04" size="1.778" layer="95" rot="R90"/>
 </segment>
 </net>
@@
 <segment>
 <pinref part="DRIVER" gate="P" pin="GND"/>
-<wire x1="-1455.42" y1="825.5" x2="-1452.88" y2="825.5" width="0.1524" layer="91"/>
+<wire x1="-1455.42" y1="822.96" x2="-1452.88" y2="825.5" width="0.1524" layer="91"/>
 <wire x1="-1452.88" y1="825.5" x2="-1452.88" y2="833.12" width="0.1524" layer="91"/>
 <pinref part="PWR" gate="G$1" pin="2"/>
 <wire x1="-1452.88" y1="833.12" x2="-1465.58" y2="833.12" width="0.1524" layer="91"/>
 <wire x1="-1465.58" y1="833.12" x2="-1465.58" y2="835.66" width="0.1524" layer="91"/>
-</segment>
-</net>
+<label x="-1450.34" y="828.04" size="1.778" layer="95" rot="R90"/>
+</segment>
+</net>

Commit message: version 2 of the board
Parts:
- removed N1: IN-16, russian-nixies:IN-16
- added NX: IN-14, russian-nixies:IN-14
Connections:
- net LHDP: now also NX.LHDP; no longer N1.LHDP
- net N$1: now also NX.9; no longer N1.9
- net N$10: now also NX.0; no longer N1.0
- net N$11: now also NX.A; no longer N1.A
- net N$2: now also NX.8; no longer N1.8
- net N$3: now also NX.7; no longer N1.7
- net N$4: now also NX.6; no longer N1.6
- net N$5: now also NX.5; no longer N1.5
- net N$6: now also NX.4; no longer N1.4
- net N$7: now also NX.3; no longer N1.3
- net N$8: now also NX.2; no longer N1.2
- net N$9: now also NX.1; no longer N1.1
- net RHDP: now also NX.RHDP; no longer N1.RHDP
Changed lines of the file:
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@@
 </classes>
 <parts>
-<part name="N1" library="russian-nixies" deviceset="IN-16" device=""/>
 <part name="DRIVER" library="74xx-us" deviceset="74*141" device="N"/>
 <part name="R1" library="SparkFun-Passives" deviceset="RESISTOR" device="AXIAL-0.3" value="10k"/>
@@
 <part name="PWR" library="SparkFun-Connectors" deviceset="M02" device="LOCK" value="5V"/>
 <part name="J1" library="SparkFun-Connectors" deviceset="M04" device="LOCK" value="D"/>
+<part name="NX" library="russian-nixies" deviceset="IN-14" device=""/>
 </parts>
 <sheets>
@@
 </plain>
 <instances>
-<instance part="N1" gate="G$1" x="-1432.56" y="797.56"/>
 <instance part="DRIVER" gate="A" x="-1465.58" y="802.64"/>
 <instance part="R1" gate="G$1" x="-1404.62" y="797.56"/>
@@
 <instance part="PWR" gate="G$1" x="-1468.12" y="843.28" rot="R270"/>
 <instance part="J1" gate="G$1" x="-1503.68" y="800.1"/>
+<instance part="NX" gate="G$1" x="-1432.56" y="800.1"/>
 </instances>
 <busses>
@@
 <net name="N$1" class="0">
 <segment>
-<pinref part="N1" gate="G$1" pin="9"/>
 <pinref part="DRIVER" gate="A" pin="9"/>
 <wire x1="-1440.18" y1="789.94" x2="-1452.88" y2="789.94" width="0.1524" layer="91"/>
+<pinref part="NX" gate="G$1" pin="9"/>
 </segment>
 </net>
 <net name="N$2" class="0">
 <segment>
-<pinref part="N1" gate="G$1" pin="8"/>
 <pinref part="DRIVER" gate="A" pin="8"/>
 <wire x1="-1440.18" y1="792.48" x2="-1452.88" y2="792.48" width="0.1524" layer="91"/>
+<pinref part="NX" gate="G$1" pin="8"/>
 </segment>
 </net>
 <net name="N$3" class="0">
 <segment>
-<pinref part="N1" gate="G$1" pin="7"/>
 <pinref part="DRIVER" gate="A" pin="7"/>
 <wire x1="-1440.18" y1="795.02" x2="-1452.88" y2="795.02" width="0.1524" layer="91"/>
+<pinref part="NX" gate="G$1" pin="7"/>
 </segment>
 </net>
 <net name="N$4" class="0">
 <segment>
-<pinref part="N1" gate="G$1" pin="6"/>
 <pinref part="DRIVER" gate="A" pin="6"/>
 <wire x1="-1440.18" y1="797.56" x2="-1452.88" y2="797.56" width="0.1524" layer="91"/>
+<pinref part="NX" gate="G$1" pin="6"/>
 </segment>
 </net>
 <net name="N$5" class="0">
 <segment>
-<pinref part="N1" gate="G$1" pin="5"/>
 <pinref part="DRIVER" gate="A" pin="5"/>
 <wire x1="-1440.18" y1="800.1" x2="-1452.88" y2="800.1" width="0.1524" layer="91"/>
+<pinref part="NX" gate="G$1" pin="5"/>
 </segment>
 </net>
 <net name="N$6" class="0">
 <segment>
-<pinref part="N1" gate="G$1" pin="4"/>
 <pinref part="DRIVER" gate="A" pin="4"/>
 <wire x1="-1440.18" y1="802.64" x2="-1452.88" y2="802.64" width="0.1524" layer="91"/>
+<pinref part="NX" gate="G$1" pin="4"/>
 </segment>
 </net>
 <net name="N$7" class="0">
 <segment>
-<pinref part="N1" gate="G$1" pin="3"/>
 <pinref part="DRIVER" gate="A" pin="3"/>
 <wire x1="-1440.18" y1="805.18" x2="-1452.88" y2="805.18" width="0.1524" layer="91"/>
+<pinref part="NX" gate="G$1" pin="3"/>
 </segment>
 </net>
 <net name="N$8" class="0">
 <segment>
-<pinref part="N1" gate="G$1" pin="2"/>
 <pinref part="DRIVER" gate="A" pin="2"/>
 <wire x1="-1440.18" y1="807.72" x2="-1452.88" y2="807.72" width="0.1524" layer="91"/>
+<pinref part="NX" gate="G$1" pin="2"/>
 </segment>
 </net>
 <net name="N$9" class="0">
 <segment>
-<pinref part="N1" gate="G$1" pin="1"/>
 <pinref part="DRIVER" gate="A" pin="1"/>
 <wire x1="-1440.18" y1="810.26" x2="-1452.88" y2="810.26" width="0.1524" layer="91"/>
+<pinref part="NX" gate="G$1" pin="1"/>
 </segment>
 </net>
 <net name="N$10" class="0">
 <segment>
-<pinref part="N1" gate="G$1" pin="0"/>
 <wire x1="-1440.18" y1="787.4" x2="-1445.26" y2="787.4" width="0.1524" layer="91"/>
 <wire x1="-1445.26" y1="787.4" x2="-1445.26" y2="812.8" width="0.1524" layer="91"/>
 <pinref part="DRIVER" gate="A" pin="0"/>
 <wire x1="-1445.26" y1="812.8" x2="-1452.88" y2="812.8" width="0.1524" layer="91"/>
+<pinref part="NX" gate="G$1" pin="0"/>
 </segment>
 </net>
@@
 <segment>
 <pinref part="R1" gate="G$1" pin="1"/>
-<pinref part="N1" gate="G$1" pin="A"/>
 <wire x1="-1409.7" y1="797.56" x2="-1422.4" y2="797.56" width="0.1524" layer="91"/>
+<pinref part="NX" gate="G$1" pin="A"/>
 </segment>
 </net>
 <net name="RHDP" class="0">
 <segment>
-<pinref part="N1" gate="G$1" pin="RHDP"/>
 <pinref part="DOTS" gate="G$1" pin="2"/>
 <wire x1="-1422.4" y1="787.4" x2="-1412.24" y2="787.4" width="0.1524" layer="91"/>
 <wire x1="-1412.24" y1="787.4" x2="-1412.24" y2="815.34" width="0.1524" layer="91"/>
 <label x="-1422.4" y="784.86" size="1.778" layer="95"/>
+<pinref part="NX" gate="G$1" pin="RHDP"/>
 </segment>
 </net>
@@
 <net name="LHDP" class="0">
 <segment>
-<pinref part="N1" gate="G$1" pin="LHDP"/>
 <pinref part="DOTS" gate="G$1" pin="1"/>
 <wire x1="-1422.4" y1="810.26" x2="-1414.78" y2="810.26" width="0.1524" layer="91"/>
 <wire x1="-1414.78" y1="810.26" x2="-1414.78" y2="815.34" width="0.1524" layer="91"/>
 <label x="-1422.4" y="807.72" size="1.778" layer="95"/>
+<pinref part="NX" gate="G$1" pin="LHDP"/>
 </segment>
 </net>
